File: Hardware/Capacitive_Touch_Keyboard.brd (EAGLE design)
At the start: 170.2 x 68.6 mm, 40 parts, among them J1 AVR_SPI_PRG_6PTH, U3 ATMEGA328P_PDIP_EZ

Commit message: v05, next proto ready for review
Parts:
- added JP1: (no value), SparkFun-Passives:SJ_2S-NO
- R1, R17, R18, R19, R20, R21, R3, R4, R5, R6, R7, R8, R9: value 1M -> 2M
- moved LED2 1.27 mm to (166.4, 39.4)
- moved BAT2 1.27 mm to (134.6, 44.5)
- moved R12 1.27 mm to (162.6, 33.0)
Connections:
- new net JP3.3: JP1.2, JP9.4
- net 3.3V: now also JP1.1; no longer JP9.4
Routing:
- net GND: track 265.9 -> 1706.6 mm
- net JP3.3: track 0.00 -> 9.53 mm
- net SCK: track 102.4 -> 94.6 mm
- net 3.3V: track 255.9 -> 248.8 mm
- net A0: track 72.9 -> 70.7 mm
- net A2: track 113.4 -> 114.8 mm
- net N$3: track 15.2 -> 16.5 mm
- net D6: track 37.3 -> 36.5 mm, vias 1 -> 2
- net MOSI: track 76.9 -> 76.2 mm, vias 1 -> 2
- net A1: track 95.6 -> 96.2 mm
Other:
- board text added: "FTDI 3.3V"
- board text added: "v05"
- board text removed: "v04"

Commit message: v10 ready for review
Parts:
- moved R6 2.84 mm to (74.9, 25.4)
- moved R1 2.54 mm to (8.89, 25.4)
- moved R11 2.54 mm to (6.35, 39.4)
- moved R14 2.54 mm to (8.89, 59.7)
- moved R17 2.54 mm to (52.1, 25.4)
- moved R19 2.54 mm to (96.5, 25.4)
- moved R20 2.54 mm to (118.1, 25.4)
- moved R3 2.54 mm to (30.5, 25.4)
- moved R8 2.54 mm to (139.7, 25.4)
- moved R9 2.54 mm to (161.3, 25.4)
- moved S2 2.54 mm to (6.35, 52.1)
- moved LED2 1.27 mm to (166.4, 40.6)
- moved LOGO1 1.27 mm to (132.7, 31.5)
- moved R12 1.27 mm to (162.6, 34.3)
Routing:
- net GND: track 1706.6 -> 1373.9 mm
- net N$16: track 0.00 -> 43.2 mm
- net N$19: track 0.00 -> 33.7 mm
- net N$11: track 0.00 -> 29.8 mm
- net N$9: track 0.00 -> 29.8 mm
- net N$6: track 0.00 -> 19.7 mm
- net N$17: track 0.00 -> 18.4 mm
- net N$13: track 0.00 -> 18.4 mm
- net N$2: track 0.00 -> 18.4 mm
- net N$21: track 0.00 -> 18.4 mm
- net N$20: track 0.00 -> 14.6 mm
- net N$14: track 0.00 -> 14.6 mm
- net N$4: track 0.00 -> 14.6 mm
- net N$8: track 0.00 -> 12.1 mm
- net N$7: track 0.00 -> 12.1 mm
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Other:
- board text added: "Gram Piano"
- board text added: "The Capacitive Touch Keyboard"
- board text added: "v10"
- board text removed: "Capacitive Touch Keyboard"
- board text removed: "v05"
