File: Hardware/Capacitive_Touch_Keyboard.sch (EAGLE design)
At the start: 47 parts, among them J1 AVR_SPI_PRG_6PTH, U2 MC34063DIP, U3 ATMEGA328P_PDIP_EZ, Y1 16MHz

Commit message: Updated resistor packages for v03
Parts:
- R12, R13: device SparkFun-Resistors:RESISTORKIT -> SparkFun-Resistors:RESISTORPTH-1/4W
Changed lines of the file:
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@@
 <part name="U2" library="SparkFun-PowerIC" deviceset="MC34063" device="DIP"/>
 <part name="R11" library="SparkFun-Resistors" deviceset="RESISTOR" device="PTH-1/4W" value="10K"/>
-<part name="R12" library="SparkFun-Resistors" deviceset="RESISTOR" device="KIT" value="3.3K"/>
-<part name="R13" library="SparkFun-Resistors" deviceset="RESISTOR" device="KIT" value="180"/>
+<part name="R12" library="SparkFun-Resistors" deviceset="RESISTOR" device="PTH-1/4W" value="3.3K"/>
+<part name="R13" library="SparkFun-Resistors" deviceset="RESISTOR" device="PTH-1/4W" value="180"/>
 <part name="R16" library="SparkFun-Resistors" deviceset="RESISTOR" device="PTH-1/4W" value="0.27"/>
 <part name="D2" library="SparkFun-DiscreteSemi" deviceset="DIODE" device="PTH" value="MBRA140"/>

Commit message: Updated inductor package for v03
Parts:
- L2: value 220 uH .86A -> 220 uH .44A; device SparkFun-Passives:INDUCTORAXIAL-0.6 -> SparkFun-Passives:INDUCTORRLB0912
Changed lines of the file:
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@@
 <part name="GND14" library="SparkFun" deviceset="GND" device=""/>
 <part name="GND18" library="SparkFun" deviceset="GND" device=""/>
-<part name="L2" library="SparkFun-Passives" deviceset="INDUCTOR" device="AXIAL-0.6" value="220 uH .86A"/>
+<part name="L2" library="SparkFun-Passives" deviceset="INDUCTOR" device="RLB0912" value="220 uH .44A"/>
 <part name="U3" library="SparkFun-DigitalIC" deviceset="ATMEGA328P_PDIP_EZ" device=""/>
 <part name="R17" library="SparkFun-Resistors" deviceset="RESISTOR" device="PTH-1/4W" value="1M"/>

Commit message: v04 protos, ready for review
Parts:
- removed C17: 1000pF, SparkFun-Capacitors:CAPKIT
- removed C19: 0.1uF, SparkFun-Capacitors:CAPKIT
- removed C4: 220uF, SparkFun-Capacitors:CAP_POLPTH1
- removed D2: MBRA140, SparkFun-DiscreteSemi:DIODEPTH
- removed JP1: (no value), SparkFun-Connectors:M02JST-PTH-2-KIT
- removed L2: 220 uH .44A, SparkFun-Passives:INDUCTORRLB0912
- removed R13: 180, SparkFun-Resistors:RESISTORPTH-1/4W
- removed R16: 0.27, SparkFun-Resistors:RESISTORPTH-1/4W
- removed SG2: BUZZER, SparkFun-Electromechanical:BUZZERPTH
- removed U2: MC34063DIP, SparkFun-PowerIC:MC34063DIP
- removed Y1: 16MHz, SparkFun-FreqCtrl:RESONATORPTH
- added BAT1, BAT2: (no value), SparkFun-Electromechanical:BATTERYAA-KIT
- added LED2: Red, SparkFun-LED:LED5MM-KIT
- added SP1: SPEAKERPCB_MOUNT, SparkFun-Electromechanical:SPEAKERPCB_MOUNT
- R11: value 10K -> TRIMPOT-PTH-KNOB; device SparkFun-Resistors:RESISTORPTH-1/4W -> SparkFun-Electromechanical:TRIMPOT-PTH-KNOB
- R12: value 3.3K -> 330
Connections:
- removed net 5V: C10.1, C19.1, C3.2, C4.+, D2.C, J1.2, JP9.VCC, R11.2, R14.2, R2.2, U3.AVCC, U3.VCC
- removed net BUZZER: SG2.1, U3.PD5(T1)
- removed net N$2: U3.PB6(XTAL1/TOSC1), Y1.1
- removed net N$677: D2.A, L2.2, U2.SWC
- removed net N$678: L2.1, R13.2, R16.2, U2.SEN
- removed net N$679: R13.1, U2.DVR
- removed net N$680: R11.1, R12.2, U2.COMP
- removed net N$681: C17.1, U2.TC
- removed net RAW_IN: R16.1, S1.S, U2.VCC
- removed net SW_VBATT: JP1.2, S1.P
- new net 3.3V: C10.1, C3.2, J1.2, JP9.VCC, LED2.A, R11.CW, R14.2, R2.2, S1.S, U3.AVCC, U3.VCC
- new net BUTTON: R14.1, S2.1, S2.2, U3.PB6(XTAL1/TOSC1)
- new net N$3: BAT1.-, BAT2.+
- new net SPEAKER: SP1.+, U3.PD5(T1)
- new net VBATT: BAT1.+, S1.P
- net A3: now also R11.WIPER; no longer R14.1, S2.1, S2.2
- net DTR: no longer J1.5
- net GND: now also BAT2.-, R11.CCW, SP1.-; no longer C17.2, C19.2, C4.-, JP1.1, SG2.2, U2.GND, U2.SWE, Y1.2
- net N$1: now also LED2.C, R12.2; no longer U3.PB7(XTAL2/TOSC2), Y1.3
- net RESET: now also J1.5
Other:
- note added: "10k Trimpot"
- moved on the sheet: C1, J1, JP9, LED1, R10, R12, R14, S2

Commit message: v05, next proto ready for review
Parts:
- added JP1: (no value), SparkFun-Passives:JUMPER-2SMD-NO
- R1, R17, R18, R19, R20, R21, R3, R4, R5, R6, R7, R8, R9: value 1M -> 2M
Connections:
- new net JP3.3: JP1.2, JP9.VCC
- net 3.3V: now also JP1.1; no longer JP9.VCC
Other:
- moved on the sheet: JP9
Changed lines of the file:
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@@
 <?xml version="1.0" encoding="utf-8"?>
 <!DOCTYPE eagle SYSTEM "eagle.dtd">
-<eagle version="6.2">
+<eagle version="6.5.0">
 <drawing>
 <settings>
@@
 <part name="P+3" library="SparkFun-Aesthetics" deviceset="3.3V" device=""/>
 <part name="J1" library="SparkFun-Connectors" deviceset="AVR_SPI_PRG_6" device="PTH"/>
-<part name="R4" library="SparkFun-Resistors" deviceset="RESISTOR" device="PTH-1/4W" value="1M"/>
-<part name="R1" library="SparkFun-Resistors" deviceset="RESISTOR" device="PTH-1/4W" value="1M"/>
+<part name="R4" library="SparkFun-Resistors" deviceset="RESISTOR" device="PTH-1/4W" value="2M"/>
+<part name="R1" library="SparkFun-Resistors" deviceset="RESISTOR" device="PTH-1/4W" value="2M"/>
 <part name="P+1" library="SparkFun-Aesthetics" deviceset="3.3V" device=""/>
 <part name="GND2" library="SparkFun-Aesthetics" deviceset="GND" device=""/>
-<part name="R3" library="SparkFun-Resistors" deviceset="RESISTOR" device="PTH-1/4W" value="1M"/>
-<part name="R5" library="SparkFun-Resistors" deviceset="RESISTOR" device="PTH-1/4W" value="1M"/>
-<part name="R6" library="SparkFun-Resistors" deviceset="RESISTOR" device="PTH-1/4W" value="1M"/>
-<part name="R7" library="SparkFun-Resistors" deviceset="RESISTOR" device="PTH-1/4W" value="1M"/>
-<part name="R8" library="SparkFun-Resistors" deviceset="RESISTOR" device="PTH-1/4W" value="1M"/>
-<part name="R9" library="SparkFun-Resistors" deviceset="RESISTOR" device="PTH-1/4W" value="1M"/>
+<part name="R3" library="SparkFun-Resistors" deviceset="RESISTOR" device="PTH-1/4W" value="2M"/>
+<part name="R5" library="SparkFun-Resistors" deviceset="RESISTOR" device="PTH-1/4W" value="2M"/>
+<part name="R6" library="SparkFun-Resistors" deviceset="RESISTOR" device="PTH-1/4W" value="2M"/>
+<part name="R7" library="SparkFun-Resistors" deviceset="RESISTOR" device="PTH-1/4W" value="2M"/>
+<part name="R8" library="SparkFun-Resistors" deviceset="RESISTOR" device="PTH-1/4W" value="2M"/>
+<part name="R9" library="SparkFun-Resistors" deviceset="RESISTOR" device="PTH-1/4W" value="2M"/>
 <part name="LOGO1" library="SparkFun-Aesthetics" deviceset="LOGO-SFE" device="NEW"/>
 <part name="LOGO2" library="SparkFun-Aesthetics" deviceset="LOGO-SFE" device="NEW"/>
 <part name="U3" library="SparkFun-DigitalIC" deviceset="ATMEGA328P_PDIP_EZ" device=""/>
-<part name="R17" library="SparkFun-Resistors" deviceset="RESISTOR" device="PTH-1/4W" value="1M"/>
-<part name="R18" library="SparkFun-Resistors" deviceset="RESISTOR" device="PTH-1/4W" value="1M"/>
-<part name="R19" library="SparkFun-Resistors" deviceset="RESISTOR" device="PTH-1/4W" value="1M"/>
-<part name="R20" library="SparkFun-Resistors" deviceset="RESISTOR" device="PTH-1/4W" value="1M"/>
-<part name="R21" library="SparkFun-Resistors" deviceset="RESISTOR" device="PTH-1/4W" value="1M"/>
+<part name="R17" library="SparkFun-Resistors" deviceset="RESISTOR" device="PTH-1/4W" value="2M"/>
+<part name="R18" library="SparkFun-Resistors" deviceset="RESISTOR" device="PTH-1/4W" value="2M"/>
+<part name="R19" library="SparkFun-Resistors" deviceset="RESISTOR" device="PTH-1/4W" value="2M"/>
+<part name="R20" library="SparkFun-Resistors" deviceset="RESISTOR" device="PTH-1/4W" value="2M"/>
+<part name="R21" library="SparkFun-Resistors" deviceset="RESISTOR" device="PTH-1/4W" value="2M"/>
 <part name="GND16" library="SparkFun" deviceset="GND" device=""/>
 <part name="S1" library="SparkFun-Electromechanical" deviceset="SWITCH-SPDT" device="KIT"/>
@@
 <part name="R12" library="SparkFun-Resistors" deviceset="RESISTOR" device="PTH-1/4W" value="330"/>
 <part name="GND8" library="SparkFun" deviceset="GND" device=""/>
+<part name="JP1" library="SparkFun-Passives" deviceset="JUMPER-2" device="SMD-NO"/>
 </parts>
 <sheets>
@@
 <instance part="GND7" gate="1" x="35.56" y="60.96"/>
 <instance part="C2" gate="G$1" x="27.94" y="81.28" rot="R90"/>
-<instance part="JP9" gate="G$1" x="104.14" y="154.94" rot="MR180"/>
+<instance part="JP9" gate="G$1" x="88.9" y="154.94" rot="MR180"/>
 <instance part="GND9" gate="1" x="48.26" y="20.32"/>
 <instance part="P+5" gate="G$1" x="35.56" y="96.52"/>
@@
 <instance part="R12" gate="G$1" x="55.88" y="132.08" rot="R90"/>
 <instance part="GND8" gate="1" x="55.88" y="121.92" rot="MR0"/>
+<instance part="JP1" gate="A" x="111.76" y="154.94" rot="R90"/>
 </instances>
 <busses>
@@
 </segment>
 <segment>
-<wire x1="109.22" y1="149.86" x2="111.76" y2="149.86" width="0.1524" layer="91"/>
+<wire x1="93.98" y1="149.86" x2="96.52" y2="149.86" width="0.1524" layer="91"/>
 <pinref part="JP9" gate="G$1" pin="CTS"/>
-<label x="111.76" y="149.86" size="1.27" layer="95" xref="yes"/>
-</segment>
-<segment>
-<wire x1="109.22" y1="147.32" x2="111.76" y2="147.32" width="0.1524" layer="91"/>
+<label x="96.52" y="149.86" size="1.27" layer="95" xref="yes"/>
+</segment>
+<segment>
+<wire x1="93.98" y1="147.32" x2="96.52" y2="147.32" width="0.1524" layer="91"/>
 <pinref part="JP9" gate="G$1" pin="GND"/>
-<label x="111.76" y="147.32" size="1.27" layer="95" xref="yes"/>
+<label x="96.52" y="147.32" size="1.27" layer="95" xref="yes"/>
 </segment>
 <segment>
@@
 <net name="RX-I" class="0">
 <segment>
-<wire x1="109.22" y1="154.94" x2="111.76" y2="154.94" width="0.1524" layer="91"/>
+<wire x1="93.98" y1="154.94" x2="96.52" y2="154.94" width="0.1524" layer="91"/>
 <pinref part="JP9" gate="G$1" pin="TXO"/>
-<label x="111.76" y="154.94" size="1.27" layer="95" xref="yes"/>
+<label x="96.52" y="154.94" size="1.27" layer="95" xref="yes"/>
 </segment>
 <segment>
@@
 <net name="TX-O" class="0">
 <segment>
-<wire x1="109.22" y1="157.48" x2="111.76" y2="157.48" width="0.1524" layer="91"/>
+<wire x1="93.98" y1="157.48" x2="96.52" y2="157.48" width="0.1524" layer="91"/>
 <pinref part="JP9" gate="G$1" pin="RXI"/>
-<label x="111.76" y="157.48" size="1.27" layer="95" xref="yes"/>
+<label x="96.52" y="157.48" size="1.27" layer="95" xref="yes"/>
 </segment>
 <segment>
@@
 <net name="DTR" class="0">
 <segment>
-<wire x1="109.22" y1="160.02" x2="111.76" y2="160.02" width="0.1524" layer="91"/>
+<wire x1="93.98" y1="160.02" x2="96.52" y2="160.02" width="0.1524" layer="91"/>
 <pinref part="JP9" gate="G$1" pin="DTR"/>
-<label x="111.76" y="160.02" size="1.27" layer="95" xref="yes"/>
+<label x="96.52" y="160.02" size="1.27" layer="95" xref="yes"/>
 </segment>
 <segment>
@@
 <net name="3.3V" class="0">
 <segment>
-<wire x1="109.22" y1="152.4" x2="111.76" y2="152.4" width="0.1524" layer="91"/>
-<pinref part="JP9" gate="G$1" pin="VCC"/>
-<label x="111.76" y="152.4" size="1.27" layer="95" xref="yes"/>
-</segment>
-<segment>
 <pinref part="J1" gate="G$1" pin="2"/>
 <wire x1="160.02" y1="154.94" x2="162.56" y2="154.94" width="0.1524" layer="91"/>
@@
 <wire x1="99.06" y1="114.3" x2="99.06" y2="116.84" width="0.1524" layer="91"/>
 </segment>
+<segment>
+<pinref part="JP1" gate="A" pin="1"/>
+<wire x1="114.3" y1="154.94" x2="116.84" y2="154.94" width="0.1524" layer="91"/>
+<label x="116.84" y="154.94" size="1.27" layer="95" xref="yes"/>
+</segment>
 </net>
 <net name="N$1" class="0">
@@
 </segment>
 </net>
+<net name="JP3.3" class="0">
+<segment>
+<pinref part="JP1" gate="A" pin="2"/>
+<wire x1="114.3" y1="157.48" x2="116.84" y2="157.48" width="0.1524" layer="91"/>
+<label x="116.84" y="157.48" size="1.27" layer="95" xref="yes"/>
+</segment>
+<segment>
+<wire x1="93.98" y1="152.4" x2="96.52" y2="152.4" width="0.1524" layer="91"/>
+<pinref part="JP9" gate="G$1" pin="VCC"/>
+<label x="96.52" y="152.4" size="1.27" layer="95" xref="yes"/>
+</segment>
+</net>

Commit message: v10 ready for review
Changed lines of the file:
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@@
 </segment>
 <segment>
-<wire x1="226.06" y1="81.28" x2="215.9" y2="81.28" width="0.1524" layer="91"/>
-<label x="220.98" y="81.28" size="1.778" layer="95"/>
+<wire x1="223.52" y1="81.28" x2="215.9" y2="81.28" width="0.1524" layer="91"/>
 <pinref part="R20" gate="G$1" pin="2"/>
+<label x="223.52" y="81.28" size="1.27" layer="95" xref="yes"/>
 </segment>
 </net>
@@
 </segment>
 <segment>
-<wire x1="226.06" y1="91.44" x2="215.9" y2="91.44" width="0.1524" layer="91"/>
-<label x="220.98" y="91.44" size="1.778" layer="95"/>
+<wire x1="223.52" y1="91.44" x2="215.9" y2="91.44" width="0.1524" layer="91"/>
 <pinref part="R21" gate="G$1" pin="2"/>
+<label x="223.52" y="91.44" size="1.27" layer="95" xref="yes"/>
 </segment>
 </net>
@@
 </segment>
 <segment>
-<wire x1="226.06" y1="101.6" x2="215.9" y2="101.6" width="0.1524" layer="91"/>
-<label x="220.98" y="101.6" size="1.778" layer="95"/>
+<wire x1="223.52" y1="101.6" x2="215.9" y2="101.6" width="0.1524" layer="91"/>
 <pinref part="R19" gate="G$1" pin="2"/>
+<label x="223.52" y="101.6" size="1.27" layer="95" xref="yes"/>
 </segment>
 </net>
@@
 </segment>
 <segment>
-<wire x1="226.06" y1="152.4" x2="215.9" y2="152.4" width="0.1524" layer="91"/>
-<label x="220.98" y="152.4" size="1.778" layer="95"/>
+<wire x1="223.52" y1="152.4" x2="215.9" y2="152.4" width="0.1524" layer="91"/>
 <pinref part="R3" gate="G$1" pin="2"/>
+<label x="223.52" y="152.4" size="1.27" layer="95" xref="yes"/>
 </segment>
 </net>
@@
 </segment>
 <segment>
-<wire x1="226.06" y1="111.76" x2="215.9" y2="111.76" width="0.1524" layer="91"/>
-<label x="220.98" y="111.76" size="1.778" layer="95"/>
+<wire x1="223.52" y1="111.76" x2="215.9" y2="111.76" width="0.1524" layer="91"/>
 <pinref part="R18" gate="G$1" pin="2"/>
+<label x="223.52" y="111.76" size="1.27" layer="95" xref="yes"/>
 </segment>
 </net>
@@
 </segment>
 <segment>
-<wire x1="226.06" y1="121.92" x2="215.9" y2="121.92" width="0.1524" layer="91"/>
-<label x="220.98" y="121.92" size="1.778" layer="95"/>
+<wire x1="223.52" y1="121.92" x2="215.9" y2="121.92" width="0.1524" layer="91"/>
 <pinref part="R6" gate="G$1" pin="2"/>
+<label x="223.52" y="121.92" size="1.27" layer="95" xref="yes"/>
 </segment>
 </net>
@@
 </segment>
 <segment>
-<wire x1="226.06" y1="132.08" x2="215.9" y2="132.08" width="0.1524" layer="91"/>
-<label x="220.98" y="132.08" size="1.778" layer="95"/>
+<wire x1="223.52" y1="132.08" x2="215.9" y2="132.08" width="0.1524" layer="91"/>
 <pinref part="R17" gate="G$1" pin="2"/>
+<label x="223.52" y="132.08" size="1.27" layer="95" xref="yes"/>
 </segment>
 </net>
@@
 </segment>
 <segment>
-<wire x1="226.06" y1="142.24" x2="215.9" y2="142.24" width="0.1524" layer="91"/>
-<label x="220.98" y="142.24" size="1.778" layer="95"/>
+<wire x1="223.52" y1="142.24" x2="215.9" y2="142.24" width="0.1524" layer="91"/>
 <pinref part="R5" gate="G$1" pin="2"/>
+<label x="223.52" y="142.24" size="1.27" layer="95" xref="yes"/>
 </segment>
 </net>
@@
 </segment>
 <segment>
-<wire x1="226.06" y1="172.72" x2="215.9" y2="172.72" width="0.1524" layer="91"/>
-<label x="220.98" y="172.72" size="1.778" layer="95"/>
+<wire x1="223.52" y1="172.72" x2="215.9" y2="172.72" width="0.1524" layer="91"/>
 <pinref part="R1" gate="G$1" pin="2"/>
+<label x="223.52" y="172.72" size="1.27" layer="95" xref="yes"/>
 </segment>
 </net>
@@
 </segment>
 <segment>
-<wire x1="226.06" y1="71.12" x2="215.9" y2="71.12" width="0.1524" layer="91"/>
-<label x="220.98" y="71.12" size="1.778" layer="95"/>
+<wire x1="223.52" y1="71.12" x2="215.9" y2="71.12" width="0.1524" layer="91"/>
 <pinref part="R7" gate="G$1" pin="2"/>
+<label x="223.52" y="71.12" size="1.27" layer="95" xref="yes"/>
 </segment>
 </net>
@@
 </segment>
 <segment>
-<wire x1="226.06" y1="60.96" x2="215.9" y2="60.96" width="0.1524" layer="91"/>
-<label x="220.98" y="60.96" size="1.778" layer="95"/>
+<wire x1="223.52" y1="60.96" x2="215.9" y2="60.96" width="0.1524" layer="91"/>
 <pinref part="R8" gate="G$1" pin="2"/>
+<label x="223.52" y="60.96" size="1.27" layer="95" xref="yes"/>
 </segment>
 </net>
@@
 </segment>
 <segment>
-<wire x1="226.06" y1="50.8" x2="215.9" y2="50.8" width="0.1524" layer="91"/>
-<label x="220.98" y="50.8" size="1.778" layer="95"/>
+<wire x1="223.52" y1="50.8" x2="215.9" y2="50.8" width="0.1524" layer="91"/>
 <pinref part="R9" gate="G$1" pin="2"/>
+<label x="223.52" y="50.8" size="1.27" layer="95" xref="yes"/>
 </segment>
 </net>
@@
 </segment>
 <segment>
-<wire x1="226.06" y1="162.56" x2="215.9" y2="162.56" width="0.1524" layer="91"/>
-<label x="220.98" y="162.56" size="1.778" layer="95"/>
+<wire x1="223.52" y1="162.56" x2="215.9" y2="162.56" width="0.1524" layer="91"/>
 <pinref part="R4" gate="G$1" pin="2"/>
+<label x="223.52" y="162.56" size="1.27" layer="95" xref="yes"/>
 </segment>
 </net>
@@
 <segment>
 <wire x1="205.74" y1="172.72" x2="198.12" y2="172.72" width="0.1524" layer="91"/>
-<label x="198.12" y="172.72" size="1.778" layer="95"/>
 <pinref part="R1" gate="G$1" pin="1"/>
+<label x="198.12" y="172.72" size="1.27" layer="95" rot="R180" xref="yes"/>
 </segment>
 <segment>
 <wire x1="205.74" y1="162.56" x2="198.12" y2="162.56" width="0.1524" layer="91"/>
-<label x="198.12" y="162.56" size="1.778" layer="95"/>
 <pinref part="R4" gate="G$1" pin="1"/>
+<label x="198.12" y="162.56" size="1.27" layer="95" rot="R180" xref="yes"/>
 </segment>
 <segment>
 <wire x1="205.74" y1="152.4" x2="198.12" y2="152.4" width="0.1524" layer="91"/>
-<label x="198.12" y="152.4" size="1.778" layer="95"/>
 <pinref part="R3" gate="G$1" pin="1"/>
+<label x="198.12" y="152.4" size="1.27" layer="95" rot="R180" xref="yes"/>
 </segment>
 <segment>
 <wire x1="205.74" y1="142.24" x2="198.12" y2="142.24" width="0.1524" layer="91"/>
-<label x="198.12" y="142.24" size="1.778" layer="95"/>
 <pinref part="R5" gate="G$1" pin="1"/>
+<label x="198.12" y="142.24" size="1.27" layer="95" rot="R180" xref="yes"/>
 </segment>
 <segment>
 <wire x1="205.74" y1="121.92" x2="198.12" y2="121.92" width="0.1524" layer="91"/>
-<label x="198.12" y="121.92" size="1.778" layer="95"/>
 <pinref part="R6" gate="G$1" pin="1"/>
+<label x="198.12" y="121.92" size="1.27" layer="95" rot="R180" xref="yes"/>
 </segment>
 <segment>
 <wire x1="205.74" y1="71.12" x2="198.12" y2="71.12" width="0.1524" layer="91"/>
-<label x="198.12" y="71.12" size="1.778" layer="95"/>
 <pinref part="R7" gate="G$1" pin="1"/>
+<label x="198.12" y="71.12" size="1.27" layer="95" rot="R180" xref="yes"/>
 </segment>
 <segment>
 <wire x1="205.74" y1="60.96" x2="198.12" y2="60.96" width="0.1524" layer="91"/>
-<label x="198.12" y="60.96" size="1.778" layer="95"/>
 <pinref part="R8" gate="G$1" pin="1"/>
+<label x="198.12" y="60.96" size="1.27" layer="95" rot="R180" xref="yes"/>
 </segment>
 <segment>
 <wire x1="205.74" y1="50.8" x2="198.12" y2="50.8" width="0.1524" layer="91"/>
-<label x="198.12" y="50.8" size="1.778" layer="95"/>
 <pinref part="R9" gate="G$1" pin="1"/>
+<label x="198.12" y="50.8" size="1.27" layer="95" rot="R180" xref="yes"/>
 </segment>
 <segment>
 <wire x1="205.74" y1="132.08" x2="198.12" y2="132.08" width="0.1524" layer="91"/>
-<label x="198.12" y="132.08" size="1.778" layer="95"/>
 <pinref part="R17" gate="G$1" pin="1"/>
+<label x="198.12" y="132.08" size="1.27" layer="95" rot="R180" xref="yes"/>
 </segment>
 <segment>
 <wire x1="205.74" y1="111.76" x2="198.12" y2="111.76" width="0.1524" layer="91"/>
-<label x="198.12" y="111.76" size="1.778" layer="95"/>
 <pinref part="R18" gate="G$1" pin="1"/>
+<label x="198.12" y="111.76" size="1.27" layer="95" rot="R180" xref="yes"/>
 </segment>
 <segment>
 <wire x1="205.74" y1="101.6" x2="198.12" y2="101.6" width="0.1524" layer="91"/>
-<label x="198.12" y="101.6" size="1.778" layer="95"/>
 <pinref part="R19" gate="G$1" pin="1"/>
+<label x="198.12" y="101.6" size="1.27" layer="95" rot="R180" xref="yes"/>
 </segment>
 <segment>
 <wire x1="205.74" y1="81.28" x2="198.12" y2="81.28" width="0.1524" layer="91"/>
-<label x="198.12" y="81.28" size="1.778" layer="95"/>
 <pinref part="R20" gate="G$1" pin="1"/>
+<label x="198.12" y="81.28" size="1.27" layer="95" rot="R180" xref="yes"/>
 </segment>
 <segment>
 <wire x1="205.74" y1="91.44" x2="198.12" y2="91.44" width="0.1524" layer="91"/>
-<label x="198.12" y="91.44" size="1.778" layer="95"/>
 <pinref part="R21" gate="G$1" pin="1"/>
-</segment>
-</net>
+<label x="198.12" y="91.44" size="1.27" layer="95" rot="R180" xref="yes"/>
+</segment>
+</net>
