File: Hardware/Gram Piano.sch (EAGLE design)
At the start: 41 parts, among them J1 AVR_SPI_PRG_6PTH, U3 ATMEGA328P_PDIP_EZ

Commit message: Added silk art
Connections:
- new net N$2: U3.PB7(XTAL2/TOSC2)
Changed lines of the file:
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@@
+</segment>
+</net>
+<net name="N$2" class="0">
+<segment>
+<pinref part="U3" gate="G$1" pin="PB7(XTAL2/TOSC2)"/>
+<wire x1="50.8" y1="50.8" x2="45.72" y2="50.8" width="0.2032" layer="91"/>
 </segment>
 </net>
